File: PCB project/Matrix USB OTG.kicad_sch (KiCad schematic)
At the start: 0 parts

Commit message: Add library
Parts:
- added J1: USB3150-30-130-A, Matrix-USB-OTG:USB3150-30-130-A_GCC, symbol Matrix-USB-OTG:USB3150-30-130-A
- added J2: SSM-102-L-DV, Matrix-USB-OTG:SAMTEC_SSM-102-L-DV, symbol Matrix-USB-OTG:SSM-102-L-DV
Connections:
- new net GND: J1.10 (GND), J1.11 (GND), J1.5 (GND), J1.6 (GND), J1.7 (GND), J1.8 (GND), J1.9 (GND), J2.04
- new net USB_DN: J1.2 (D-), J2.01
- new net USB_DP: J1.3 (D+), J2.03
- new net VBUS: J1.1 (VBUS), J2.02
- no-connect marks 0 -> 1
Other:
- note added: "ID pin needs to be left floating as it will work as device."

Commit message: Final schematic and initial constraints
Connections:
- net GND: now also J2.03; no longer J2.04
- net USB_DN: now also J2.02; no longer J2.01
- net USB_DP: now also J2.01; no longer J2.03
- net VBUS: now also J2.04; no longer J2.02
Other:
- moved on the sheet: J2

Commit message: Make the PCB smaller so it can work with ESQ-105-23-T-D
Parts:
- J1: value USB3150-30-130-A -> USB3150-30-70-A; footprint Matrix-USB-OTG:USB3150-30-130-A_GCC -> USB3150-30-70-A_GCC
Changed lines of the file:
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@@
 	)
 	(image
-		(at 92.71 49.53)
+		(at 80.01 40.64)
+		(scale 0.261131)
 		(data "iVBORw0KGgoAAAANSUhEUgAAB4AAAAQICAYAAADsqcbuAAAABHNCSVQICAgIfAhkiAAAIABJREFU"
 			"eJzs3Xl8VNX5+PHPnS2TPSEhKxASIIQQdmhA0KKIoEhxqVj1hyxWtFa/trgXFBCtKC1WpRZRQepS"
@@
 			)
 		)
-		(property "Value" "USB3150-30-130-A"
+		(property "Value" "USB3150-30-70-A"
 			(at 151.13 102.87 0)
 			(show_name no)
@@
 			)
 		)
-		(property "Footprint" "Matrix-USB-OTG:USB3150-30-130-A_GCC"
+		(property "Footprint" "USB3150-30-70-A_GCC"
 			(at 140.97 102.616 0)
 			(hide yes)

Commit message: Fix USB footprint issues and change the pcb width to 0.8mm as per USB 3150 datasheet
Parts:
- J1: footprint USB3150-30-70-A_GCC -> Matrix-USB-OTG:USB3150-30-130-A_GCC
Connections:
- net GND: no longer J1.10 (GND), J1.11 (GND)
Changed lines of the file:
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@@
 	)
 	(junction
-		(at 130.81 123.19)
-		(diameter 0)
-		(color 0 0 0 0)
-	)
-	(junction
 		(at 125.73 101.6)
 		(diameter 0)
@@
 	(wire
 		(pts
-			(xy 130.81 123.19) (xy 133.35 123.19)
-		)
-		(stroke
-			(width 0)
-			(type default)
-		)
-	)
-	(wire
-		(pts
 			(xy 208.28 111.76) (xy 208.28 116.84)
 		)
@@
 			)
 		)
-		(property "Footprint" "USB3150-30-70-A_GCC"
+		(property "Footprint" "Matrix-USB-OTG:USB3150-30-130-A_GCC"
 			(at 140.97 102.616 0)
 			(hide yes)
@@
 		(pin "6"
 		)
-		(pin "10"
-		)
-		(pin "11"
-		)
 		(pin "5"
