File: PCB project/Matrix USB OTG.kicad_sch (KiCad schematic)
At the start: 2 parts, among them J1 USB3150-30-70-A, J2 SSM-102-L-DV

Commit message: Final check and adjustments before generating manufacturing files
Parts:
- J1: value USB3150-30-70-A -> USB3150-30-130-A; Digikey PN (none) -> 2073-USB3150-30-130-ACT-ND - Cut Tape (CT); MANUFACTURER (none) -> GCT
- J2: Digikey PN (none) -> 612-SSM-102-L-DV-ND; RS PN (none) -> 765-5351P
Connections:
- net GND: now also J1.10 (GND), J1.11 (GND)
Changed lines of the file:
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@@
 	)
 	(junction
+		(at 130.81 123.19)
+		(diameter 0)
+		(color 0 0 0 0)
+	)
+	(junction
 		(at 128.27 123.19)
 		(diameter 0)
@@
 	(wire
 		(pts
+			(xy 130.81 123.19) (xy 133.35 123.19)
+		)
+		(stroke
+			(width 0)
+			(type default)
+		)
+	)
+	(wire
+		(pts
 			(xy 181.61 111.76) (xy 181.61 114.3)
 		)
@@
 			)
 		)
-		(property "Value" "USB3150-30-70-A"
+		(property "Value" "USB3150-30-130-A"
 			(at 151.13 102.87 0)
 			(show_name no)
@@
 			)
 		)
-		(property "Datasheet" "USB3150-30-130-A"
+		(property "Datasheet" "https://gct.co/files/specs/usb3150-spec.pdf"
 			(at 138.684 102.362 0)
 			(hide yes)
@@
 			)
 		)
-		(property "Description" ""
+		(property "Description" "USB - micro B USB 2.0 Plug Connector 5 Position Through Hole"
 			(at 105.41 90.17 0)
 			(hide yes)
@@
 			)
 		)
-		(property "Digikey PN" ""
+		(property "Digikey PN" "2073-USB3150-30-130-ACT-ND - Cut Tape (CT)"
+			(at 105.41 90.17 0)
+			(hide yes)
+			(show_name no)
+			(do_not_autoplace no)
+			(effects
+				(font
+					(size 1.27 1.27)
+				)
+			)
+		)
+		(property "MANUFACTURER" "GCT"
 			(at 105.41 90.17 0)
 			(hide yes)
@@
 		(pin "1"
 		)
+		(pin "11"
+		)
+		(pin "10"
+		)
 		(instances
 			(project "Matrix USB OTG"
@@
 			)
 		)
-		(property "Datasheet" ""
+		(property "Datasheet" "https://suddendocs.samtec.com/catalog_english/ssm_sm.pdf?_gl"
 			(at 195.58 111.76 0)
 			(hide yes)
@@
 			)
 		)
-		(property "Description" ""
+		(property "Description" "4 Position Receptacle, Pass Through Connector 0.100\" (2.54mm) Surface Mount Gold"
 			(at 195.58 111.76 0)
 			(hide yes)
@@
 			)
 		)
-		(property "RS PN" ""
+		(property "RS PN" "765-5351P"
 			(at 195.58 111.76 0)
 			(hide yes)
@@
 			)
 		)
-		(property "Digikey PN" ""
+		(property "Digikey PN" "612-SSM-102-L-DV-ND"
 			(at 195.58 111.76 0)
 			(hide yes)

Commit message: Manufacturing package V1
Parts:
- added FID1, FID2, FID3: Fiducial, Fiducial:Fiducial_0.5mm_Mask1.5mm, symbol Mechanical:Fiducial
