File: PCB project/Matrix USB OTG.kicad_pcb (KiCad board)
At the start: 4 copper layers, 20.2 x 16.4 mm, 2 parts, among them J1 USB3150-30-70-A, J2 SSM-102-L-DV

Commit message: Final check and adjustments before generating manufacturing files
Parts:
- J1: value USB3150-30-70-A -> USB3150-30-130-A
- moved J1 75.2 mm to (196.3, 128.7)
- moved J2 75.2 mm to (187.2, 116.8)
Routing:
- net GND: vias 4 -> 15
