File: PCB project/Matrix USB OTG.kicad_pcb (KiCad board)
At the start: 4 copper layers, 20.2 x 16.4 mm, 2 parts, among them J1 USB3150-30-130-A, J2 SSM-102-L-DV

Commit message: Manufacturing package V1
Parts:
- added FID1: Fiducial, Fiducial:Fiducial_0.5mm_Mask1.5mm, F.Cu at (182.8, 120.8)
- added FID2: Fiducial, Fiducial:Fiducial_0.5mm_Mask1.5mm, F.Cu at (189.2, 129.9)
- added FID3: Fiducial, Fiducial:Fiducial_0.5mm_Mask1.5mm, F.Cu at (200.3, 126.5)
Routing:
- net VBUS: track 4.91 -> 4.00 mm, vias 4 -> 3
- net GND: vias 15 -> 13
